Commit message: 部署 dog3 步态策略：相位可配 + 模型与训练端对齐
- rl_controller：步态相位速率由硬编码 π/2 改为可配（gait_period），
  与训练端 gait_phase 的 cycle_time 对应；相位观测无需再改 C++
- controllers.yaml：num_obs 45→51、observations_name 增加 "phases"、
  gait_period: 1.0、joint_kp/kd 40/1.0
- URDF/xacro：与 dog3lab 保持完全一致（关节 origin/limit 平移、后足原位）
- 策略 ONNX 更新为最新训练结果
- 新增 tools/bag2csv.py（rosbag2 → CSV，供 PlotJuggler 分析）
- README 重写：编译、启动、键位、部署新策略、模型约定、数据记录

Gazebo 中可正常站立/行走/转向，站立姿态左右对称。

File: urdfs/dog3_description/urdf/dog3.urdf (robot description, URDF)
Before this commit: robot dog3, 18 links, 17 joints
Joints:
- joint LH_FOOT_joint: origin xyz=-0.0965776536 -0.03089611695 -0.2449908695 rpy=0 0 0 -> xyz=-0.06157765364946 -0.03089611695 -0.2449908695 rpy=0 0 0
- joint RH_FOOT_joint: origin xyz=-0.0968978639 0.03015880125 -0.2425423888 rpy=0 0 0 -> xyz=-0.06189786389862 0.03015880125 -0.2425423888 rpy=0 0 0

File: urdfs/dog3_description/xacro/robot.xacro (robot description, xacro)
@@ -366,5 +366,5 @@
   </link>
   <joint name="LH_FOOT_joint" type="fixed">
-    <origin xyz="-0.0965776536 -0.03089611695 -0.2449908695" rpy="0 0 0" />
+    <origin xyz="-0.06157765364946 -0.03089611695 -0.2449908695" rpy="0 0 0" />
     <parent link="RL_calf" />
     <child link="LH_FOOT" />
@@ -481,5 +481,5 @@
   </link>
   <joint name="RH_FOOT_joint" type="fixed">
-    <origin xyz="-0.0968978639 0.03015880125 -0.2425423888" rpy="0 0 0" />
+    <origin xyz="-0.06189786389862 0.03015880125 -0.2425423888" rpy="0 0 0" />
     <parent link="RR_calf" />
     <child link="RH_FOOT" />
